File: receiving end.sch (EAGLE design)
At the start: 19 parts, among them IC1 MEGA8-P, IC2 74LS125D, IC3 NUD4001, IC4 NUD4001, IC5 NUD4001, Q1 16 MHz

Commit message: polished schematic
Parts:
- removed C1: 22 pF, rcl:C-EUC1206
- removed C2: 22pF, rcl:C-EUC1206
- removed IC2: 74LS125D, 74xx-eu:74LS125D
- removed IC3, IC4, IC5: NUD4001, led:NUD4001
- removed Q1: 16 MHz, crystal:MC-405
- removed R3, R4, R5: 1.4 ohm, resistor:R-EU_R0805
- removed S1: SWS001, smd-special:SWS001
- added T2: (no value), solomon_library:PMOSSOT23ZXM61P02FTA
- T1, T3: device zetex:NMOS2SM8 -> solomon_library:PMOSSOT23ZXM61P02FTA
Connections:
- removed net BRAKE_LEDS: IC5.IOUT
- removed net LEFT_LEDS: IC4.IOUT
- removed net N$13: IC3.REXT, R4.2
- removed net N$14: IC4.BOOST, T1B.S
- removed net N$34: IC4.REXT, R3.2
- removed net N$36: IC5.REXT, R5.2
- removed net N$37: IC3.BOOST, T1A.S
- removed net RIGHT_LEDS: IC3.IOUT
- net GND: now also IC1.PB6(XTAL1/TOSC1), IC1.PB7(XTAL2/TOSC2); no longer C1.1, C2.1, IC2A.OE, IC2B.OE, IC2C.OE, IC2D.I, IC2D.O, IC2D.OE, IC2P.GND, IC3.GND, IC4.GND, IC5.GND, T1A.D, T1B.D, T3A.D
- net N$1: now also T2.S; no longer C2.2, IC1.PB6(XTAL1/TOSC1), Q1.2
- net N$10: now also T2.G; no longer IC2B.I
- net N$11: now also T1.G; no longer IC2A.I
- net N$2: now also T3.S; no longer C1.2, IC1.PB7(XTAL2/TOSC2), Q1.1
- net N$25: now also R2.2
- net N$3: now also IC1.PD5(T1); no longer IC2C.O, T3A.G
- net N$35: no longer S1.1
- net N$5: now also T3.D; no longer IC1.PD5(T1), R2.2
- net N$6: now also T2.D; no longer IC2B.O, T1B.G
- net N$7: now also T1.D; no longer IC5.BOOST, T3A.S
- net N$8: now also T1.S; no longer IC2A.O, T1A.G
- net N$9: now also T3.G; no longer IC2C.I
- net VCC: no longer IC2P.VCC, IC3.VIN, IC4.VIN, IC5.VIN, R3.1, R4.1, R5.1, S1.2
Other:
- note removed: "NIGHT RIDER Abdullah Madan Brandon Valentine Jesse Bates Solomon Cooper"
- moved on the sheet: R1

Commit message: eceiving end schematic before making the changes that Andrew suggested
Parts:
- removed T3: (no value), solomon_library:PMOSSOT23ZXM61P02FTA
- added G1, G2: AB9V, battery:AB9V
- added LMP1, LMP2: (no value), special:LAMP
- added R3, R5: 0, resistor:R-EU_R0805
Connections:
- removed net N$1 (its old number): T2.S
- new net N$10: LMP2.2, R5.2
- net GND: now also G1.-
- net N$2: now also IC1.PC3(ADC3); no longer T3.S
- net N$5: now also LMP1.1, T1.D; no longer T3.D
- net N$6: now also LMP1.2, R3.2; no longer T2.D
- net N$7: now also LMP2.1, T2.D; no longer T1.D
- net N$8: now also G2.-, T2.S
- net N$9: now also G2.+, R3.1, R5.1; no longer IC1.PC3(ADC3), T3.G
- net VCC: now also G1.+
Other:
- moved on the sheet: T1, T2
Changed lines of the file:
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@@
 <layer number="48" name="Document" color="7" fill="1" visible="yes" active="no"/>
 <layer number="49" name="Reference" color="7" fill="1" visible="yes" active="no"/>
-<layer number="51" name="tDocu" color="6" fill="9" visible="yes" active="no"/>
+<layer number="51" name="tDocu" color="7" fill="1" visible="yes" active="no"/>
 <layer number="52" name="bDocu" color="7" fill="1" visible="yes" active="no"/>
 <layer number="91" name="Nets" color="2" fill="1" visible="yes" active="yes"/>
@@
 <part name="T1" library="solomon_library" deviceset="PMOSSOT23" device="ZXM61P02FTA"/>
 <part name="T2" library="solomon_library" deviceset="PMOSSOT23" device="ZXM61P02FTA"/>
-<part name="T3" library="solomon_library" deviceset="PMOSSOT23" device="ZXM61P02FTA"/>
+<part name="G1" library="battery" deviceset="AB9V" device=""/>
+<part name="SUPPLY1" library="supply2" deviceset="GND" device=""/>
+<part name="LMP1" library="special" deviceset="LAMP" device=""/>
+<part name="LMP2" library="special" deviceset="LAMP" device=""/>
+<part name="G2" library="battery" deviceset="AB9V" device=""/>
+<part name="R3" library="resistor" deviceset="R-EU_" device="R0805" value="0"/>
+<part name="R5" library="resistor" deviceset="R-EU_" device="R0805" value="0"/>
 </parts>
 <sheets>
@@
 <instance part="IC1" gate="G$1" x="73.66" y="50.8"/>
 <instance part="SUPPLY3" gate="GND" x="35.56" y="45.72"/>
-<instance part="SUPPLY4" gate="GND" x="38.1" y="66.04"/>
+<instance part="SUPPLY4" gate="GND" x="38.1" y="71.12"/>
 <instance part="SUPPLY6" gate="GND" x="134.62" y="48.26" rot="R270"/>
 <instance part="IR2" gate="A" x="149.86" y="43.18" rot="R180"/>
@@
 <instance part="R2" gate="G$1" x="119.38" y="43.18" rot="R180"/>
 <instance part="SUPPLY9" gate="GND" x="124.46" y="20.32"/>
-<instance part="P+4" gate="VCC" x="27.94" y="88.9"/>
+<instance part="P+4" gate="VCC" x="25.4" y="109.22"/>
 <instance part="P+5" gate="VCC" x="142.24" y="22.86"/>
 <instance part="JP1" gate="A" x="83.82" y="2.54"/>
@@
 <instance part="P+8" gate="VCC" x="27.94" y="71.12"/>
 <instance part="P+7" gate="VCC" x="38.1" y="30.48"/>
-<instance part="T1" gate="A" x="144.78" y="109.22"/>
-<instance part="T2" gate="A" x="144.78" y="91.44"/>
-<instance part="T3" gate="A" x="144.78" y="71.12"/>
+<instance part="T1" gate="A" x="114.3" y="93.98"/>
+<instance part="T2" gate="A" x="124.46" y="76.2"/>
+<instance part="G1" gate="G$1" x="38.1" y="101.6" rot="R180"/>
+<instance part="SUPPLY1" gate="GND" x="50.8" y="96.52"/>
+<instance part="LMP1" gate="G$1" x="142.24" y="104.14"/>
+<instance part="LMP2" gate="G$1" x="142.24" y="86.36"/>
+<instance part="G2" gate="G$1" x="182.88" y="99.06" rot="MR90"/>
+<instance part="R3" gate="G$1" x="160.02" y="99.06" rot="R180"/>
+<instance part="R5" gate="G$1" x="160.02" y="81.28" rot="R180"/>
 </instances>
 <busses>
@@
 <net name="GND" class="0">
 <segment>
-<pinref part="SUPPLY4" gate="GND" pin="GND"/>
-<pinref part="IC1" gate="G$1" pin="GND"/>
-<wire x1="38.1" y1="73.66" x2="50.8" y2="73.66" width="0.1524" layer="91"/>
-<wire x1="38.1" y1="73.66" x2="38.1" y2="68.58" width="0.1524" layer="91"/>
-<pinref part="IC1" gate="G$1" pin="AREF"/>
-<wire x1="50.8" y1="71.12" x2="50.8" y2="73.66" width="0.1524" layer="91"/>
-<junction x="50.8" y="73.66"/>
-</segment>
-<segment>
 <pinref part="IR2" gate="A" pin="GND"/>
 <pinref part="SUPPLY6" gate="GND" pin="GND"/>
@@
 <wire x1="50.8" y1="48.26" x2="35.56" y2="48.26" width="0.1524" layer="91"/>
 </segment>
+<segment>
+<pinref part="G1" gate="G$1" pin="-"/>
+<pinref part="SUPPLY1" gate="GND" pin="GND"/>
+<wire x1="50.8" y1="101.6" x2="50.8" y2="99.06" width="0.1524" layer="91"/>
+</segment>
+<segment>
+<pinref part="IC1" gate="G$1" pin="GND"/>
+<wire x1="38.1" y1="73.66" x2="50.8" y2="73.66" width="0.1524" layer="91"/>
+<pinref part="IC1" gate="G$1" pin="AREF"/>
+<wire x1="50.8" y1="71.12" x2="50.8" y2="73.66" width="0.1524" layer="91"/>
+<junction x="50.8" y="73.66"/>
+<pinref part="SUPPLY4" gate="GND" pin="GND"/>
+</segment>
 </net>
 <net name="N$4" class="0">
@@
 </segment>
 </net>
-<net name="N$9" class="0">
-<segment>
-<wire x1="119.38" y1="68.58" x2="119.38" y2="71.12" width="0.1524" layer="91"/>
-<pinref part="IC1" gate="G$1" pin="PC3(ADC3)"/>
-<wire x1="119.38" y1="71.12" x2="99.06" y2="71.12" width="0.1524" layer="91"/>
-<wire x1="119.38" y1="68.58" x2="139.7" y2="68.58" width="0.1524" layer="91"/>
-<pinref part="T3" gate="A" pin="G"/>
-</segment>
-</net>
-<net name="N$10" class="0">
-<segment>
-<pinref part="IC1" gate="G$1" pin="PC2(ADC2)"/>
-<wire x1="99.06" y1="73.66" x2="119.38" y2="73.66" width="0.1524" layer="91"/>
-<wire x1="119.38" y1="73.66" x2="119.38" y2="88.9" width="0.1524" layer="91"/>
-<wire x1="119.38" y1="88.9" x2="139.7" y2="88.9" width="0.1524" layer="91"/>
-<pinref part="T2" gate="A" pin="G"/>
-</segment>
-</net>
 <net name="N$11" class="0">
 <segment>
 <pinref part="IC1" gate="G$1" pin="PC1(ADC1)"/>
-<wire x1="99.06" y1="76.2" x2="116.84" y2="76.2" width="0.1524" layer="91"/>
-<wire x1="116.84" y1="76.2" x2="116.84" y2="106.68" width="0.1524" layer="91"/>
-<wire x1="116.84" y1="106.68" x2="139.7" y2="106.68" width="0.1524" layer="91"/>
+<wire x1="99.06" y1="76.2" x2="109.22" y2="76.2" width="0.1524" layer="91"/>
 <pinref part="T1" gate="A" pin="G"/>
+<wire x1="109.22" y1="76.2" x2="109.22" y2="91.44" width="0.1524" layer="91"/>
 </segment>
 </net>
@@
 </segment>
 <segment>
-<pinref part="P+4" gate="VCC" pin="VCC"/>
-<wire x1="35.56" y1="78.74" x2="27.94" y2="78.74" width="0.1524" layer="91"/>
-<wire x1="27.94" y1="78.74" x2="27.94" y2="86.36" width="0.1524" layer="91"/>
-<junction x="35.56" y="78.74"/>
-</segment>
-<segment>
 <pinref part="JP1" gate="A" pin="2"/>
 <wire x1="88.9" y1="5.08" x2="99.06" y2="5.08" width="0.1524" layer="91"/>
@@
 <pinref part="P+7" gate="VCC" pin="VCC"/>
 <wire x1="50.8" y1="27.94" x2="38.1" y2="27.94" width="0.1524" layer="91"/>
+</segment>
+<segment>
+<pinref part="G1" gate="G$1" pin="+"/>
+<pinref part="P+4" gate="VCC" pin="VCC"/>
+<wire x1="25.4" y1="101.6" x2="25.4" y2="106.68" width="0.1524" layer="91"/>
 </segment>
 </net>
@@
 </segment>
 </net>
+<net name="N$1" class="0">
+<segment>
+<pinref part="IC1" gate="G$1" pin="PC2(ADC2)"/>
+<pinref part="T2" gate="A" pin="G"/>
+<wire x1="99.06" y1="73.66" x2="119.38" y2="73.66" width="0.1524" layer="91"/>
+</segment>
+</net>
+<net name="N$2" class="0">
+<segment>
+<pinref part="IC1" gate="G$1" pin="PC3(ADC3)"/>
+<junction x="99.06" y="71.12"/>
+</segment>
+</net>
 <net name="N$5" class="0">
 <segment>
-<wire x1="160.02" y1="76.2" x2="144.78" y2="76.2" width="0.1524" layer="91"/>
-<junction x="160.02" y="76.2"/>
-<pinref part="T3" gate="A" pin="D"/>
+<pinref part="T1" gate="A" pin="D"/>
+<wire x1="114.3" y1="99.06" x2="142.24" y2="99.06" width="0.1524" layer="91"/>
+<pinref part="LMP1" gate="G$1" pin="1"/>
+</segment>
+</net>
+<net name="N$7" class="0">
+<segment>
+<pinref part="T2" gate="A" pin="D"/>
+<wire x1="124.46" y1="81.28" x2="142.24" y2="81.28" width="0.1524" layer="91"/>
+<pinref part="LMP2" gate="G$1" pin="1"/>
+</segment>
+</net>
+<net name="N$8" class="0">
+<segment>
+<pinref part="G2" gate="G$1" pin="-"/>
+<pinref part="T1" gate="A" pin="S"/>
+<wire x1="182.88" y1="86.36" x2="180.34" y2="86.36" width="0.1524" layer="91"/>
+<wire x1="180.34" y1="86.36" x2="114.3" y2="86.36" width="0.1524" layer="91"/>
+<wire x1="114.3" y1="86.36" x2="114.3" y2="88.9" width="0.1524" layer="91"/>
+<pinref part="T2" gate="A" pin="S"/>
+<wire x1="124.46" y1="71.12" x2="180.34" y2="71.12" width="0.1524" layer="91"/>
+<wire x1="180.34" y1="71.12" x2="180.34" y2="86.36" width="0.1524" layer="91"/>
+<junction x="180.34" y="86.36"/>
+</segment>
+</net>
+<net name="N$9" class="0">
+<segment>
+<wire x1="165.1" y1="99.06" x2="170.18" y2="99.06" width="0.1524" layer="91"/>
+<pinref part="R3" gate="G$1" pin="1"/>
+<pinref part="G2" gate="G$1" pin="+"/>
+<wire x1="182.88" y1="111.76" x2="170.18" y2="111.76" width="0.1524" layer="91"/>
+<wire x1="170.18" y1="111.76" x2="170.18" y2="99.06" width="0.1524" layer="91"/>
+<pinref part="R5" gate="G$1" pin="1"/>
+<wire x1="165.1" y1="81.28" x2="170.18" y2="81.28" width="0.1524" layer="91"/>
+<wire x1="170.18" y1="81.28" x2="170.18" y2="99.06" width="0.1524" layer="91"/>
+<junction x="170.18" y="99.06"/>
 </segment>
 </net>
 <net name="N$6" class="0">
 <segment>
-<wire x1="162.56" y1="96.52" x2="144.78" y2="96.52" width="0.1524" layer="91"/>
-<junction x="162.56" y="96.52"/>
-<pinref part="T2" gate="A" pin="D"/>
-</segment>
-</net>
-<net name="N$7" class="0">
-<segment>
-<wire x1="162.56" y1="114.3" x2="144.78" y2="114.3" width="0.1524" layer="91"/>
-<junction x="162.56" y="114.3"/>
-<pinref part="T1" gate="A" pin="D"/>
-</segment>
-</net>
-<net name="N$2" class="0">
-<segment>
-<wire x1="144.78" y1="66.04" x2="172.72" y2="66.04" width="0.1524" layer="91"/>
-<junction x="172.72" y="66.04"/>
-<pinref part="T3" gate="A" pin="S"/>
-</segment>
-</net>
-<net name="N$1" class="0">
-<segment>
-<wire x1="144.78" y1="86.36" x2="172.72" y2="86.36" width="0.1524" layer="91"/>
-<junction x="172.72" y="86.36"/>
-<pinref part="T2" gate="A" pin="S"/>
-</segment>
-</net>
-<net name="N$8" class="0">
-<segment>
-<wire x1="144.78" y1="104.14" x2="172.72" y2="104.14" width="0.1524" layer="91"/>
-<junction x="172.72" y="104.14"/>
-<pinref part="T1" gate="A" pin="S"/>
+<pinref part="R3" gate="G$1" pin="2"/>
+<pinref part="LMP1" gate="G$1" pin="2"/>
+<wire x1="144.78" y1="99.06" x2="154.94" y2="99.06" width="0.1524" layer="91"/>
+</segment>
+</net>
+<net name="N$10" class="0">
+<segment>
+<pinref part="R5" gate="G$1" pin="2"/>
+<pinref part="LMP2" gate="G$1" pin="2"/>
+<wire x1="144.78" y1="81.28" x2="154.94" y2="81.28" width="0.1524" layer="91"/>
 </segment>
 </net>
@@
 </sheet>
 </sheets>
+<errors>
+</errors>
 </schematic>
 </drawing>
